Commit message: Add files via upload

File: ur5_no1.urdf (robot description, URDF)
Before this commit: robot ur5, 9 links, 8 joints
Links:
- removed link base_inertia
- added link base
Joints:
- removed joint base_to_base_inertia
- added joint base_link-base_fixed_joint: type fixed, parent base_link, child base, origin xyz=0 0 0 rpy=0 0 0
- joint ee_fixed_joint: origin xyz=0.0 0.0823 0.0 rpy=0.0 0.0 1.570796327 -> xyz=0 0.0823 0.0 rpy=0 0 1.57079
- joint elbow_joint: origin xyz=0.0 0.1197 0.42500 rpy=0.0 0.0 0.0 -> xyz=0.0 -0.1197 0.42500 rpy=0.0 0.0 0.0
- joint shoulder_pan_joint: parent base_inertia -> base_link
- joint wrist_2_joint: limit lower=-3.141592 upper=3.141592 effort=28.0 velocity=3.2 -> lower=-3.1415 upper=3.1415 effort=28.0 velocity=3.2; origin xyz=0.0 0.093 0.0 rpy=0.0 0.0 0.0 -> xyz=0.0 0.093 0.0 rpy=0 0 0
- joint wrist_3_joint: limit lower=-3.141592 upper=3.141592 effort=28.0 velocity=3.2 -> lower=-3.1415 upper=3.1415 effort=28.0 velocity=3.2; origin xyz=0.0 0.0 0.09465 rpy=0.0 0.0 0.0 -> xyz=0.0 0.0 0.09465 rpy=0 0 0
